File: pcb/decopling.kicad_sch (KiCad schematic)
At the start: 24 parts

Commit message: refactor(pcb): strip down
Connections:
- net P1.35V is gone; now on net P3.3V: C62.1, C64.1, C66.1, C68.1
Changed lines of the file:
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@@
 		)
 	)
-	(global_label "P1.35V"
+	(global_label "P3.3V"
 		(shape passive)
 		(at 124.46 60.96 90)
@@
 		)
 	)
-	(global_label "P1.35V"
+	(global_label "P3.3V"
 		(shape passive)
 		(at 102.87 60.96 90)
