File: pcb/fileFPGA.kicad_sch (KiCad schematic)
At the start: 13 parts, among them J6 JTAG, U3 LFE5U-25F-8MG285C, U6 W25Q128JVP

Commit message: refactor(pcb): strip down
Parts:
- removed C1, C19, C25: 10nF, Capacitor_SMD:C_0201_0603Metric, symbol Device:C
- removed C20, C26, C4: 100nF, Capacitor_SMD:C_0201_0603Metric, symbol Device:C
Connections:
- net P3.3V: now also U3.G14 (VCCIO7[2]), U3.G5 (VCCIO2[2]), U3.H14 (VCCIO7[2]), U3.H5 (VCCIO2[2]), U3.M14 (VCCIO6[2]), U3.N14 (VCCIO6[2])
- net ADC_CTRL0: no longer names the net of U3.G1 (PR32B)
- net ADC_CTRL1: no longer names the net of U3.F1 (PR35C)
- net ADC_MUX0: no longer names the net of U3.F4 (PR26C/PCLKT3_0)
- net ADC_MUX1: no longer names the net of U3.F3 (PR26D/PCLKC3_0)
- net ADC_MUX2: no longer names the net of U3.F2 (PR32A)
- net ADC_MUX3: no longer names the net of U3.H1 (PR35D)
- net ADC_SENSE_HI: no longer names the net of U3.H3 (PR29A/GR_PCLK3_0)
- net ADC_SENSE_LO: no longer names the net of U3.G3 (PR29B)
- removed net ECP5_VREF: U3.B4 (PR14C/VREF1_2), U3.C15 (PL14C/VREF1_7), U3.H15 (PL35B/VREF1_6)
- net EXT_PLL+: no longer names the net of U3.M16 (PL47C/LLC_GPLL0T_IN)
- net EXT_PLL-: no longer names the net of U3.M17 (PL47D/LLC_GPLL0C_IN)
- net IO_0: no longer names the net of U3.N17 (PB6A/D5/MISO2/IO5)
- net IO_1: no longer names the net of U3.M18 (PB6B/D4/MOSI2/IO4)
- net IO_10: no longer names the net of U3.B8 (PT67A)
- net IO_11: no longer names the net of U3.A8 (PT35B/PCLKC1_0)
- net IO_12: no longer names the net of U3.H2 (PR29D)
- net IO_13: no longer names the net of U3.J2 (PR35A)
- net IO_5: no longer names the net of U3.B10 (PT29A/PCLKT0_0)
- net IO_6: no longer names the net of U3.B9 (PT33A/PCLKT1_1)
- net IO_9: no longer names the net of U3.C8 (PT67B)
- net IO_A0: no longer names the net of U3.L4 (PR38B)
- net IO_A1: no longer names the net of U3.N3 (PR38D)
- net IO_A2: no longer names the net of U3.N4 (PR38C)
- net IO_A3: no longer names the net of U3.H4 (PR26A/PCLKT3_1)
- net IO_A4: no longer names the net of U3.G4 (PR26B/PCLKC3_1)
- net IO_A5: no longer names the net of U3.T17 (PB13B/CS1N)
- net IO_MISO: no longer names the net of U3.N15 (PB4A/D7/IO7)
- net IO_MOSI: no longer names the net of U3.N16 (PB4B/D6/IO6)
- net IO_SCK: no longer names the net of U3.R17 (PB13A/SN/CSN)
- net IO_SCL: no longer names the net of U3.C9 (PT33B/PCLKC1_1)
- net IO_SDA: no longer names the net of U3.C10 (PT29B/PCLKC0_0)
- removed net P1.35V: U3.B18 (PL23C/PCLKT7_0), U3.C6 (PR5B), U3.D17 (PL26A/PCLKT6_1), U3.G14 (VCCIO7[2]), U3.G5 (VCCIO2[2]), U3.H14 (VCCIO7[2]), U3.H5 (VCCIO2[2]), U3.K15 (PL41D), U3.K16 (PL41C), U3.K17 (PL44A), U3.M14 (VCCIO6[2]), U3.N14 (VCCIO6[2])
- net RAM_A0: no longer names the net of U3.C4 (PR14B)
- net RAM_A1: no longer names the net of U3.D2 (PR23A/PCLKT2_1)
- net RAM_A10: no longer names the net of U3.A7 (PR8B)
- net RAM_A11: no longer names the net of U3.C2 (PR17B)
- net RAM_A12: no longer names the net of U3.B6 (PR8A)
- net RAM_A13: no longer names the net of U3.C1 (PR23C/PCLKT2_0)
- net RAM_A14: no longer names the net of U3.A2 (PR20C/GR_PCLK2_0)
- net RAM_A15: no longer names the net of U3.C7 (PR2A)
- net RAM_A2: no longer names the net of U3.D3 (PR17A)
- net RAM_A3: no longer names the net of U3.A3 (PR20A/GR_PCLK2_1)
- net RAM_A4: no longer names the net of U3.A4 (PR11B)
- net RAM_A5: no longer names the net of U3.D4 (PR14A)
- net RAM_A6: no longer names the net of U3.C3 (PR14D)
- net RAM_A7: no longer names the net of U3.B2 (PR20B)
- net RAM_A8: no longer names the net of U3.B1 (PR23B/PCLKC2_1)
- net RAM_A9: no longer names the net of U3.D1 (PR23D/PCLKC2_0)
- net RAM_BA0: no longer names the net of U3.D6 (PR5A)
- net RAM_BA1: no longer names the net of U3.B7 (PR2B/S0_IN)
- net RAM_BA2: no longer names the net of U3.A6 (PR11A)
- net RAM_CAS#: no longer names the net of U3.D13 (PL8A)
- net RAM_CK+: no longer names the net of U3.J18 (PL41A)
- net RAM_CK-: no longer names the net of U3.K18 (PL41B)
- net RAM_CKE: no longer names the net of U3.D18 (PL26C/PCLKT6_0)
- net RAM_CS#: no longer names the net of U3.A12 (PL5A)
- net RAM_D0: no longer names the net of U3.C17 (PL23D/PCLKC7_0)
- net RAM_D1: no longer names the net of U3.D15 (PL17A)
- net RAM_D10: no longer names the net of U3.G15 (PL35A)
- net RAM_D11: no longer names the net of U3.F15 (PL29C/GR_PCLK6_1)
- net RAM_D12: no longer names the net of U3.J16 (PL35D)
- net RAM_D13: no longer names the net of U3.C18 (PL26B/PCLKC6_1)
- net RAM_D14: no longer names the net of U3.H16 (PL35C)
- net RAM_D15: no longer names the net of U3.F18 (PL26D/PCLKC6_0)
- net RAM_D2: no longer names the net of U3.B17 (PL23B/PCLKC7_1)
- net RAM_D3: no longer names the net of U3.C16 (PL20C/GR_PCLK7_0)
- net RAM_D4: no longer names the net of U3.A15 (PL14D)
- net RAM_D5: no longer names the net of U3.B13 (PL14A)
- net RAM_D6: no longer names the net of U3.A17 (PL23A/PCLKT7_1)
- net RAM_D7: no longer names the net of U3.A13 (PL14B)
- net RAM_D8: no longer names the net of U3.F17 (PL29A/GR_PCLK6_0)
- net RAM_D9: no longer names the net of U3.F16 (PL29B)
- net RAM_LDM: no longer names the net of U3.G16 (PL29D)
- net RAM_LDQS+: no longer names the net of U3.G18 (PL32A)
- net RAM_LDQS-: no longer names the net of U3.H17 (PL32B)
- net RAM_ODT: no longer names the net of U3.C13 (PL8B)
- net RAM_RAS#: no longer names the net of U3.C12 (PL2A)
- net RAM_RESET#: no longer names the net of U3.L18 (PL44B)
- net RAM_UDM: no longer names the net of U3.D16 (PL17B)
- net RAM_UDQS+: no longer names the net of U3.B15 (PL20A/GR_PCLK7_1)
- net RAM_UDQS-: no longer names the net of U3.A16 (PL20B)
- net RAM_WE#: no longer names the net of U3.B12 (PL2B)
- net SPI_0: no longer names the net of U3.A10 (PT27B/PCLKC0_1)
- net SPI_1: no longer names the net of U3.C11 (PT4B)
- net SPI_2: no longer names the net of U3.A11 (PT27A/PCLKT0_1)
- net SPI_3: no longer names the net of U3.B11 (PT4A)
- net USER_BUTTON: no longer names the net of U3.J17 (PL38C)
- no-connect marks 6 -> 101
